Commit message: update b2w,go2w.

File: loco_manipulation_gym/resources/robots/go2w/urdf/go2w.urdf (robot description, URDF)
Before this commit: robot go2w_description, 33 links, 32 joints
Links:
- link FL_calf: geometry collision cylinder length=0.12 radius=0.012; visual mesh filename=../dae/calf.dae
- link FR_calf: geometry collision cylinder length=0.12 radius=0.013; visual mesh filename=../dae/calf_mirror.dae
- link RL_calf: geometry collision cylinder length=0.12 radius=0.013; visual mesh filename=../dae/calf.dae
- link RR_calf: geometry collision cylinder length=0.12 radius=0.013; visual mesh filename=../dae/calf_mirror.dae
